Commit message: Phase 2 (WIP): complex layout, walking people, battery sim, energy-aware manager, people tracker, collision monitor, test scenarios
- tunibot_gazebo_plugins: HumanActorPlugin (animated actor + lidar-visible collision body, yields to the robot)
- world v2 (scripts/build_world.py): kitchen behind a 0.9 m door, 1.05 m service corridor with L-turn,
  VIP lounge behind a third doorway, 4 walking people, closed exterior door, gazebo_ros_state
- auto_mapping.launch.py + auto_mapper: autonomous Cartographer mapping tour
- battery_simulator: physics-based power model, CC-CV charging on dock contact, learned Wh/m
- delivery_manager v2: energy-aware order planning from Nav2 path lengths, return-to-dock before
  depletion, alternate approach poses, BLOCKED detection, docking with contact check, e-stop
- people_tracker: lidar clustering + Kalman tracking, predicted-motion cost mask, social speed limit
- navigation.launch.py: own Nav2 bringup with collision_monitor, people filter, custom BT
- scenario_runner + run_tests.sh + make_test_report: 12 automated test cases with ground-truth metrics
- /clock at 100 Hz (gazebo_ros_init default 10 Hz starved the sim-time Nav2 loops)

Co-Authored-By: Claude Opus 5.5 <noreply@anthropic.com>

File: src/tunibot_delivery/urdf/waiter_robot.urdf.xacro (robot description, xacro)
@@ -126,4 +126,22 @@
     </plugin>
   </gazebo>
+  <!-- Bumper (contact sensor) on the body, spine and lidar housing: ground truth for the
+       collision metrics of the Phase 2 tests (/bumper). Fixed joints are lumped into
+       base_footprint by the URDF->SDF conversion, hence the collision names. -->
+  <gazebo reference="base_footprint">
+    <sensor name="bumper" type="contact">
+      <always_on>true</always_on>
+      <update_rate>20</update_rate>
+      <contact>
+        <collision>base_footprint_fixed_joint_lump__base_link_collision</collision>
+        <collision>base_footprint_fixed_joint_lump__back_spine_link_collision_1</collision>
+        <collision>base_footprint_fixed_joint_lump__base_scan_collision_4</collision>
+      </contact>
+      <plugin name="bumper_plugin" filename="libgazebo_ros_bumper.so">
+        <ros><remapping>bumper_states:=bumper</remapping></ros>
+        <frame_name>base_footprint</frame_name>
+      </plugin>
+    </sensor>
+  </gazebo>
   <!-- Plugin Gazebo LiDAR (Ray Sensor) -->
   <gazebo reference="base_scan">

Commit message: Phase 2: serving-window kitchen layout, corner dock, new map, robot physics and navigation fixes
Layout (per the team's restaurant concept): kitchen (staff-only keepout) hands food to the
robot through 2 serving windows; charging dock in the dining-room corner; VIP lounge via a
0.9 m door, 1.05 m corridor with recessed doors, L-turn and a third doorway. Frames: map = world + (9, -2.2).

Fixes found by testing:
- robot physics: soft wheel contact (minDepth 1 mm) let the frictionless casters carry the
  load; forward speed was 15 % of the command (also in Phase 1). Casters 4 mm smaller, stiff contact.
- world generator made every door 0.75 m instead of 0.9 m (wall end extension at door edges)
- Cartographer corridor degeneracy / perceptual aliasing: odometry-weighted correlative matching,
  bounded loop-closure search, non-identical corridor features
- Nav2 Humble: yaw goal tolerance + RPP path pruning -> 'plan has 0 poses'; heading now aligned by the manager
- collision monitor: big static stop zone froze in-place turns near walls; approach model stuttered
- people tracker: TF listener on its own node/thread; only tracks that walked 0.6 m are people;
  no detections inside the robot's own radius
- battery: charger powers the electronics + charges the pack (SoC was stuck at 97.7 %)
- delivery manager: precise docking (go-to-point + heading/lateral-corrected reverse, 0.7 cm
  from the pad centre in test), latched ERROR, motion-based BLOCKED detection, reachability
  pre-check, deliberate departure from the serving window, rclpy logger severity bug

Co-Authored-By: Claude Opus 5.5 <noreply@anthropic.com>

File: src/tunibot_delivery/urdf/waiter_robot.urdf.xacro (robot description, xacro)
@@ -50,6 +50,6 @@
   <!-- Roues folles (casters): sans elles le robot bascule et la base frotte le sol -> glissement + LiDAR incline -->
   <link name="caster_front_link">
-    <collision><geometry><sphere radius="0.039"/></geometry></collision>
-    <visual><geometry><sphere radius="0.039"/></geometry><material name="black"/></visual>
+    <collision><geometry><sphere radius="0.035"/></geometry></collision>
+    <visual><geometry><sphere radius="0.035"/></geometry><material name="black"/></visual>
     <inertial><mass value="0.1"/><inertia ixx="0.0001" ixy="0" ixz="0" iyy="0.0001" iyz="0" izz="0.0001"/></inertial>
   </link>
@@ -58,6 +58,6 @@
   </joint>
   <link name="caster_back_link">
-    <collision><geometry><sphere radius="0.039"/></geometry></collision>
-    <visual><geometry><sphere radius="0.039"/></geometry><material name="black"/></visual>
+    <collision><geometry><sphere radius="0.035"/></geometry></collision>
+    <visual><geometry><sphere radius="0.035"/></geometry><material name="black"/></visual>
     <inertial><mass value="0.1"/><inertia ixx="0.0001" ixy="0" ixz="0" iyy="0.0001" iyz="0" izz="0.0001"/></inertial>
   </link>
@@ -68,8 +68,8 @@
   <gazebo reference="caster_back_link"><mu1>0.0</mu1><mu2>0.0</mu2></gazebo>
   <gazebo reference="wheel_left_link">
-    <mu1>1.0</mu1><mu2>1.0</mu2><kp>1000000.0</kp><kd>100.0</kd><minDepth>0.001</minDepth><maxVel>0.1</maxVel><fdir1>1 0 0</fdir1>
+    <mu1>1.0</mu1><mu2>1.0</mu2><fdir1>1 0 0</fdir1>
   </gazebo>
   <gazebo reference="wheel_right_link">
-    <mu1>1.0</mu1><mu2>1.0</mu2><kp>1000000.0</kp><kd>100.0</kd><minDepth>0.001</minDepth><maxVel>0.1</maxVel><fdir1>1 0 0</fdir1>
+    <mu1>1.0</mu1><mu2>1.0</mu2><fdir1>1 0 0</fdir1>
   </gazebo>
   <!-- Support LiDAR -->
@@ -116,5 +116,5 @@
       <wheel_diameter>0.16</wheel_diameter>
       <max_wheel_torque>20</max_wheel_torque>
-      <max_wheel_acceleration>1.0</max_wheel_acceleration>
+      <max_wheel_acceleration>1.5</max_wheel_acceleration>
       <command_topic>cmd_vel</command_topic>
       <publish_odom>true</publish_odom>

Commit message: Robot model: damped stiff wheel contact + axle friction (robot drifted 15 cm / 15 deg after stopping); energy learning weights long missions
Co-Authored-By: Claude Opus 5.5 <noreply@anthropic.com>

File: src/tunibot_delivery/urdf/waiter_robot.urdf.xacro (robot description, xacro)
@@ -34,4 +34,5 @@
     <parent link="base_link"/>
     <child link="wheel_left_link"/>
+    <dynamics damping="0.2" friction="0.5"/>
     <origin xyz="0 0.22 -0.02" rpy="-1.5708 0 0"/>
     <axis xyz="0 0 1"/>
@@ -45,4 +46,5 @@
     <parent link="base_link"/>
     <child link="wheel_right_link"/>
+    <dynamics damping="0.2" friction="0.5"/>
     <origin xyz="0 -0.22 -0.02" rpy="-1.5708 0 0"/>
     <axis xyz="0 0 1"/>
@@ -50,6 +52,6 @@
   <!-- Roues folles (casters): sans elles le robot bascule et la base frotte le sol -> glissement + LiDAR incline -->
   <link name="caster_front_link">
-    <collision><geometry><sphere radius="0.035"/></geometry></collision>
-    <visual><geometry><sphere radius="0.035"/></geometry><material name="black"/></visual>
+    <collision><geometry><sphere radius="0.039"/></geometry></collision>
+    <visual><geometry><sphere radius="0.039"/></geometry><material name="black"/></visual>
     <inertial><mass value="0.1"/><inertia ixx="0.0001" ixy="0" ixz="0" iyy="0.0001" iyz="0" izz="0.0001"/></inertial>
   </link>
@@ -58,6 +60,6 @@
   </joint>
   <link name="caster_back_link">
-    <collision><geometry><sphere radius="0.035"/></geometry></collision>
-    <visual><geometry><sphere radius="0.035"/></geometry><material name="black"/></visual>
+    <collision><geometry><sphere radius="0.039"/></geometry></collision>
+    <visual><geometry><sphere radius="0.039"/></geometry><material name="black"/></visual>
     <inertial><mass value="0.1"/><inertia ixx="0.0001" ixy="0" ixz="0" iyy="0.0001" iyz="0" izz="0.0001"/></inertial>
   </link>
@@ -68,8 +70,8 @@
   <gazebo reference="caster_back_link"><mu1>0.0</mu1><mu2>0.0</mu2></gazebo>
   <gazebo reference="wheel_left_link">
-    <mu1>1.0</mu1><mu2>1.0</mu2><fdir1>1 0 0</fdir1>
+    <mu1>1.0</mu1><mu2>1.0</mu2><kp>1000000.0</kp><kd>100.0</kd><minDepth>0.0</minDepth><maxVel>0.1</maxVel><fdir1>1 0 0</fdir1>
   </gazebo>
   <gazebo reference="wheel_right_link">
-    <mu1>1.0</mu1><mu2>1.0</mu2><fdir1>1 0 0</fdir1>
+    <mu1>1.0</mu1><mu2>1.0</mu2><kp>1000000.0</kp><kd>100.0</kd><minDepth>0.0</minDepth><maxVel>0.1</maxVel><fdir1>1 0 0</fdir1>
   </gazebo>
   <!-- Support LiDAR -->
@@ -116,5 +118,5 @@
       <wheel_diameter>0.16</wheel_diameter>
       <max_wheel_torque>20</max_wheel_torque>
-      <max_wheel_acceleration>1.5</max_wheel_acceleration>
+      <max_wheel_acceleration>0.0</max_wheel_acceleration>
       <command_topic>cmd_vel</command_topic>
       <publish_odom>true</publish_odom>
